File: hardware/BREAD_Slice.kicad_pcb (KiCad board)
At the start: 2 copper layers, 70 x 100 mm, 24 parts, among them J1 I2C_01x04, J2 Conn_01x10_Female, J3 Screw_Terminal_01x02, J4 Screw_Terminal_01x02, J5 Screw_Terminal_01x02, J6 Screw_Terminal_01x02, U2 ACS723xMATR-10AB, U3 ACS723xMATR-10AB, U4 ACS723xMATR-10AB, U5 ACS723xMATR-10AB

Commit message: updated silkscreen info
Other:
- board text added: "BREAD Slice Current Reader (SLC_CRXX) Cam K Brooks rev.A [09-2024]"
- board text removed: "10/20/40A Current Slice SLC_CRxx R0 2024"
- board text removed: "BREAD Slice Template SLC_TEMP <version> <year>"
Changed lines of the file:
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@@
 		)
 	)
-	(gr_text "BREAD Slice\nTemplate\nSLC_TEMP\n<version> <year>"
-		(at 126.066 104.035 270)
+	(gr_text "BREAD Slice\nCurrent Reader\n(SLC_CRXX)\nCam K Brooks\nrev.A [09-2024]"
+		(at 127.172 103.224 270)
 		(layer "F.SilkS")
 		(effects
@@
 				(thickness 0.15)
 			)
-		)
-	)
-	(gr_text "10/20/40A Current Slice\nSLC_CRxx\nR0 2024"
-		(at 142.7 44.8 0)
-		(layer "F.SilkS")
-		(effects
-			(font
-				(size 1 1)
-				(thickness 0.15)
-			)
