File: hardware/isolated_acdc_current_sensor_acs724.kicad_sch (KiCad schematic)
At the start: 5 parts, among them U10 ACS724xLCTR-50AB

Commit message: completed board
Parts:
- C5: renamed from C21; footprint (none) -> Capacitor_SMD:C_0805_2012Metric_Pad1.18x1.45mm_HandSolder
- C6: renamed from C22; footprint (none) -> Capacitor_SMD:C_0805_2012Metric_Pad1.18x1.45mm_HandSolder
- C7: renamed from C23; footprint (none) -> Capacitor_SMD:C_0805_2012Metric_Pad1.18x1.45mm_HandSolder
- R1: renamed from R39; footprint (none) -> Resistor_SMD:R_0805_2012Metric_Pad1.20x1.40mm_HandSolder
- renumbered U10 to U2
Changed lines of the file:
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@@
 		(on_board yes)
 		(dnp no)
-		(property "Reference" "C21"
+		(property "Reference" "C5"
 			(at 115.062 106.172 0)
 			(effects
@@
 			)
 		)
-		(property "Footprint" ""
+		(property "Footprint" "Capacitor_SMD:C_0805_2012Metric_Pad1.18x1.45mm_HandSolder"
 			(at 118.4148 104.14 0)
 			(effects
@@
 		(instances
 			(project "BREAD_Slice"
-				(path "/66043bca-a260-4915-9fce-8a51d324c687/0303321c-07d5-4b3a-88db-b57740d57f62"
-					(reference "C24")
-					(unit 1)
-				)
-				(path "/66043bca-a260-4915-9fce-8a51d324c687/fb558bf0-5f57-4d6a-b949-86f12669227c"
-					(reference "C21")
+				(path "/66043bca-a260-4915-9fce-8a51d324c687/fb558bf0-5f57-4d6a-b949-86f12669227c"
+					(reference "C5")
 					(unit 1)
 				)
@@
 		(on_board yes)
 		(dnp no)
-		(property "Reference" "C23"
+		(property "Reference" "C7"
 			(at 134.112 106.172 0)
 			(effects
@@
 			)
 		)
-		(property "Footprint" ""
+		(property "Footprint" "Capacitor_SMD:C_0805_2012Metric_Pad1.18x1.45mm_HandSolder"
 			(at 137.4648 104.14 0)
 			(effects
@@
 		(instances
 			(project "BREAD_Slice"
-				(path "/66043bca-a260-4915-9fce-8a51d324c687/0303321c-07d5-4b3a-88db-b57740d57f62"
-					(reference "C26")
-					(unit 1)
-				)
-				(path "/66043bca-a260-4915-9fce-8a51d324c687/fb558bf0-5f57-4d6a-b949-86f12669227c"
-					(reference "C23")
+				(path "/66043bca-a260-4915-9fce-8a51d324c687/fb558bf0-5f57-4d6a-b949-86f12669227c"
+					(reference "C7")
 					(unit 1)
 				)
@@
 		(on_board yes)
 		(dnp no)
-		(property "Reference" "#PWR034"
+		(property "Reference" "#PWR018"
 			(at 151.13 121.92 0)
 			(effects
@@
 		(instances
 			(project "BREAD_Slice"
-				(path "/66043bca-a260-4915-9fce-8a51d324c687/0303321c-07d5-4b3a-88db-b57740d57f62"
-					(reference "#PWR036")
-					(unit 1)
-				)
-				(path "/66043bca-a260-4915-9fce-8a51d324c687/fb558bf0-5f57-4d6a-b949-86f12669227c"
-					(reference "#PWR034")
+				(path "/66043bca-a260-4915-9fce-8a51d324c687/fb558bf0-5f57-4d6a-b949-86f12669227c"
+					(reference "#PWR018")
 					(unit 1)
 				)
@@
 		(on_board yes)
 		(dnp no)
-		(property "Reference" "#PWR033"
+		(property "Reference" "#PWR017"
 			(at 138.43 96.52 0)
 			(effects
@@
 		(instances
 			(project "BREAD_Slice"
-				(path "/66043bca-a260-4915-9fce-8a51d324c687/0303321c-07d5-4b3a-88db-b57740d57f62"
-					(reference "#PWR035")
-					(unit 1)
-				)
-				(path "/66043bca-a260-4915-9fce-8a51d324c687/fb558bf0-5f57-4d6a-b949-86f12669227c"
-					(reference "#PWR033")
+				(path "/66043bca-a260-4915-9fce-8a51d324c687/fb558bf0-5f57-4d6a-b949-86f12669227c"
+					(reference "#PWR017")
 					(unit 1)
 				)
@@
 		(on_board yes)
 		(dnp no)
-		(property "Reference" "U10"
+		(property "Reference" "U2"
 			(at 155.702 88.646 0)
 			(effects
@@
 		(instances
 			(project "BREAD_Slice"
-				(path "/66043bca-a260-4915-9fce-8a51d324c687/0303321c-07d5-4b3a-88db-b57740d57f62"
-					(reference "U11")
-					(unit 1)
-				)
-				(path "/66043bca-a260-4915-9fce-8a51d324c687/fb558bf0-5f57-4d6a-b949-86f12669227c"
-					(reference "U10")
+				(path "/66043bca-a260-4915-9fce-8a51d324c687/fb558bf0-5f57-4d6a-b949-86f12669227c"
+					(reference "U2")
 					(unit 1)
 				)
@@
 		(on_board yes)
 		(dnp no)
-		(property "Reference" "C22"
+		(property "Reference" "C6"
 			(at 134.112 84.582 0)
 			(effects
@@
 			)
 		)
-		(property "Footprint" ""
+		(property "Footprint" "Capacitor_SMD:C_0805_2012Metric_Pad1.18x1.45mm_HandSolder"
 			(at 137.4648 82.55 0)
 			(effects
@@
 		(instances
 			(project "BREAD_Slice"
-				(path "/66043bca-a260-4915-9fce-8a51d324c687/0303321c-07d5-4b3a-88db-b57740d57f62"
-					(reference "C25")
-					(unit 1)
-				)
-				(path "/66043bca-a260-4915-9fce-8a51d324c687/fb558bf0-5f57-4d6a-b949-86f12669227c"
-					(reference "C22")
+				(path "/66043bca-a260-4915-9fce-8a51d324c687/fb558bf0-5f57-4d6a-b949-86f12669227c"
+					(reference "C6")
 					(unit 1)
 				)
@@
 		(on_board yes)
 		(dnp no)
-		(property "Reference" "R39"
+		(property "Reference" "R1"
 			(at 127 95.504 90)
 			(effects
@@
 			)
 		)
-		(property "Footprint" ""
+		(property "Footprint" "Resistor_SMD:R_0805_2012Metric_Pad1.20x1.40mm_HandSolder"
 			(at 127 102.108 90)
 			(effects
@@
 		(instances
 			(project "BREAD_Slice"
-				(path "/66043bca-a260-4915-9fce-8a51d324c687/0303321c-07d5-4b3a-88db-b57740d57f62"
-					(reference "R40")
-					(unit 1)
-				)
-				(path "/66043bca-a260-4915-9fce-8a51d324c687/fb558bf0-5f57-4d6a-b949-86f12669227c"
-					(reference "R39")
-					(unit 1)
-				)
+				(path "/66043bca-a260-4915-9fce-8a51d324c687/fb558bf0-5f57-4d6a-b949-86f12669227c"
+					(reference "R1")
+					(unit 1)
+				)
