File: hardware/isolated_dc_voltage_sensor.kicad_sch (KiCad schematic)
At the start: 31 parts, among them U14 TLV9001IDCK

Commit message: initial commit after split of ac and dc
Parts:
- renumbered U to U16, U to U17, U to U19
Changed lines of the file:
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@@
 		(on_board yes)
 		(dnp no)
-		(property "Reference" "U"
+		(property "Reference" "U?"
 			(at 252.476 128.778 0)
 			(effects
@@
 				(path "/66043bca-a260-4915-9fce-8a51d324c687/2d631dd3-3c2c-4fa9-892f-1ec301d37d00"
 					(reference "U19")
+					(unit 1)
+				)
+				(path "/66043bca-a260-4915-9fce-8a51d324c687/78aa2bdd-0100-4a0d-9a5e-97e57d8c85b9"
+					(reference "U?")
 					(unit 1)
 				)
@@
 		(dnp no)
 		(fields_autoplaced yes)
-		(property "Reference" "U"
+		(property "Reference" "U?"
 			(at 156.21 71.12 0)
 			(effects
@@
 				(path "/66043bca-a260-4915-9fce-8a51d324c687/2d631dd3-3c2c-4fa9-892f-1ec301d37d00"
 					(reference "U16")
+					(unit 1)
+				)
+				(path "/66043bca-a260-4915-9fce-8a51d324c687/78aa2bdd-0100-4a0d-9a5e-97e57d8c85b9"
+					(reference "U?")
 					(unit 1)
 				)
@@
 		(on_board yes)
 		(dnp no)
-		(property "Reference" "U"
+		(property "Reference" "U?"
 			(at 155.956 26.67 0)
 			(effects
@@
 					(unit 1)
 				)
+				(path "/66043bca-a260-4915-9fce-8a51d324c687/78aa2bdd-0100-4a0d-9a5e-97e57d8c85b9"
+					(reference "U?")
+					(unit 1)
+				)

Commit message: completed board
Parts:
- removed C32: 10u, symbol Device:C
- removed C33: 0.1u, symbol Device:C
- removed R47: 10k 0.1%, symbol Device:R
- added C13, C14: 10n, Capacitor_SMD:C_0603_1608Metric_Pad1.08x0.95mm_HandSolder, symbol Device:C
- added C15: 0.1u, Capacitor_SMD:C_0603_1608Metric_Pad1.08x0.95mm_HandSolder, symbol Device:C
- added C17: 10u, Capacitor_SMD:C_0603_1608Metric_Pad1.08x0.95mm_HandSolder, symbol Device:C
- added C21: 0.1u, Capacitor_SMD:C_0805_2012Metric_Pad1.18x1.45mm_HandSolder, symbol Device:C
- added R8: 10k, Resistor_SMD:R_0805_2012Metric_Pad1.20x1.40mm_HandSolder, symbol Device:R
- C10: renamed from C29; footprint (none) -> Capacitor_SMD:C_0603_1608Metric_Pad1.08x0.95mm_HandSolder
- C11: renamed from C31; footprint (none) -> Capacitor_SMD:C_0603_1608Metric_Pad1.08x0.95mm_HandSolder; Specs (none) -> X5R
- C12: renamed from C30; footprint (none) -> Capacitor_SMD:C_0603_1608Metric_Pad1.08x0.95mm_HandSolder
- C16: renamed from C34; footprint (none) -> Capacitor_SMD:C_0805_2012Metric_Pad1.18x1.45mm_HandSolder
- C18: renamed from C35; footprint (none) -> Capacitor_SMD:C_0805_2012Metric_Pad1.18x1.45mm_HandSolder
- C19: renamed from C36; footprint (none) -> Capacitor_SMD:C_0805_2012Metric_Pad1.18x1.45mm_HandSolder
- C20: renamed from C37; footprint (none) -> Capacitor_SMD:C_0805_2012Metric_Pad1.18x1.45mm_HandSolder
- C8: renamed from C27; footprint (none) -> Capacitor_SMD:C_0603_1608Metric_Pad1.08x0.95mm_HandSolder
- C9: renamed from C28; footprint (none) -> Capacitor_SMD:C_0603_1608Metric_Pad1.08x0.95mm_HandSolder; Specs (none) -> X5R
- NT2: footprint NetTie:NetTie-2_SMD_Pad2.0mm -> NetTie:NetTie-2_SMD_Pad0.5mm
- R2: renamed from R41; value 16.9k 1% -> 16.9k; footprint (none) -> Resistor_SMD:R_0603_1608Metric_Pad0.98x0.95mm_HandSolder; Specs (none) -> 1%
- R3: renamed from R42; value 10k 1% -> 10k; footprint (none) -> Resistor_SMD:R_0603_1608Metric_Pad0.98x0.95mm_HandSolder; Specs (none) -> 1%
- R4: renamed from R43; footprint (none) -> Resistor_SMD:R_0805_2012Metric_Pad1.20x1.40mm_HandSolder
- R5: renamed from R44; footprint (none) -> Resistor_SMD:R_0805_2012Metric_Pad1.20x1.40mm_HandSolder
- R6: renamed from R45; footprint (none) -> Resistor_SMD:R_0805_2012Metric_Pad1.20x1.40mm_HandSolder
- R7: renamed from R46; value 10k 0.1% -> 10k; footprint (none) -> Resistor_SMD:R_0805_2012Metric_Pad1.20x1.40mm_HandSolder; Spec (none) -> 0.1%
- R9: renamed from R48; footprint (none) -> Resistor_SMD:R_0805_2012Metric_Pad1.20x1.40mm_HandSolder
- RSNS1, RX1, RX2, RX3, RX4, RX5, RX6: footprint (none) -> Resistor_SMD:R_1206_3216Metric_Pad1.30x1.75mm_HandSolder
- U3: renamed from U16; footprint DWV0008A -> kml-custom:DWV0008A
- U4: renamed from U17; footprint RS_20_ADI -> kml-custom:RS_20_ADI
- renumbered U14 to U5, U19 to U6
Connections:
- net GND: now also C14.1, C15.1, C17.1, C21.1, R8.2
- net GNDISO: now also C13.1
- net VDD: now also C14.2, C15.2, C17.2, C21.2
- net VDD_ISO: now also C13.2; no longer R3.1
- net VSEL: now also R3.1
- net at R7.2, U5.1 (+): now also R8.1
- net ~{ISOPWR}: now reaches U4.8 (PDIS)
Other:
- note added: "Distance between low ESR bypass must be <2mm"
- moved on the sheet: C11, C9, R2, R3, R7, U5
