File: hardware/isolated_dc_voltage_sensor.kicad_sch (KiCad schematic)
At the start: 34 parts, among them U3 AMC1311BDWVR, U4 ADUM5010ARSZ-RL7, U5 TLV9001IDCK, U6 TLV9001IDCK

Commit message: fix(hw): re-point stale library nicknames
These parts exist in KiCad-Master-Lib; the boards referenced libraries that no
longer exist (kml-custom, KML-Custom, and SparkFun libraries that never
contained the part) or names the library has since changed.

KiCad embeds footprint geometry in the .kicad_pcb, so the boards rendered and
fabricated correctly and the rot stayed invisible -- it only surfaces on
update-from-library, or when a generator tries to resolve a nickname.

Nickname/name only. No geometry is changed:

  SparkFun-DiscreteSemi:AP63205 -> KMLib_IC_Power:AP63205WU-7_Buck_Regulator
  kml-custom:ADUM5010ARSZ-RL7 -> KMLib_IC_Power:ADUM5010ARSZ-RL7_Isolated_DC-DC
  kml-custom:AMC1311BDWVR -> KMLib_IC_Analog:AMC1311BDWVR_Isolation_Amplifier
  kml-custom:DWV0008A -> KMLib_IC_SMD:DWV0008A
  kml-custom:RS_20_ADI -> KMLib_IC_SMD:RS_20_ADI
  kml-custom:WAGO_2606-1104_010-000 -> KMLib_Connectors:2606-1104_010-000_Wago

Only references that failed to resolve were touched. Generic parts (<=4 pins)
and KiCad *-rescue libraries are deliberately excluded: fingerprint matching
cannot distinguish a 2-pin resistor from a 2-pin capacitor, so those are being
done by hand.
Parts:
- U3: footprint kml-custom:DWV0008A -> KMLib_IC_SMD:DWV0008A; symbol kml-custom:AMC1311BDWVR -> KMLib_IC_Analog:AMC1311BDWVR_Isolation_Amplifier
- U4: footprint kml-custom:RS_20_ADI -> KMLib_IC_SMD:RS_20_ADI; symbol kml-custom:ADUM5010ARSZ-RL7 -> KMLib_IC_Power:ADUM5010ARSZ-RL7_Isolated_DC-DC
Changed lines of the file:
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@@
 	)
 	(symbol
-		(lib_id "kml-custom:AMC1311BDWVR")
+		(lib_id "KMLib_IC_Analog:AMC1311BDWVR_Isolation_Amplifier")
 		(at 156.21 88.9 0)
 		(unit 1)
@@
 			)
 		)
-		(property "Footprint" "kml-custom:DWV0008A"
+		(property "Footprint" "KMLib_IC_SMD:DWV0008A"
 			(at 156.21 88.9 0)
 			(hide yes)
@@
 	)
 	(symbol
-		(lib_id "kml-custom:ADUM5010ARSZ-RL7")
+		(lib_id "KMLib_IC_Power:ADUM5010ARSZ-RL7_Isolated_DC-DC")
 		(at 179.07 36.83 0)
 		(mirror y)
@@
 			)
 		)
-		(property "Footprint" "kml-custom:RS_20_ADI"
+		(property "Footprint" "KMLib_IC_SMD:RS_20_ADI"
 			(at 179.07 36.83 0)
 			(hide yes)
