File: hardware/BREAD_Slice.kicad_sch (KiCad schematic)
At the start: 16 parts, among them J1 Conn_01x10_Female, J2 2606-1104/010-000, U1 AP63205

Commit message: fix(hw): re-point stale library nicknames
These parts exist in KiCad-Master-Lib; the boards referenced libraries that no
longer exist (kml-custom, KML-Custom, and SparkFun libraries that never
contained the part) or names the library has since changed.

KiCad embeds footprint geometry in the .kicad_pcb, so the boards rendered and
fabricated correctly and the rot stayed invisible -- it only surfaces on
update-from-library, or when a generator tries to resolve a nickname.

Nickname/name only. No geometry is changed:

  SparkFun-DiscreteSemi:AP63205 -> KMLib_IC_Power:AP63205WU-7_Buck_Regulator
  kml-custom:ADUM5010ARSZ-RL7 -> KMLib_IC_Power:ADUM5010ARSZ-RL7_Isolated_DC-DC
  kml-custom:AMC1311BDWVR -> KMLib_IC_Analog:AMC1311BDWVR_Isolation_Amplifier
  kml-custom:DWV0008A -> KMLib_IC_SMD:DWV0008A
  kml-custom:RS_20_ADI -> KMLib_IC_SMD:RS_20_ADI
  kml-custom:WAGO_2606-1104_010-000 -> KMLib_Connectors:2606-1104_010-000_Wago

Only references that failed to resolve were touched. Generic parts (<=4 pins)
and KiCad *-rescue libraries are deliberately excluded: fingerprint matching
cannot distinguish a 2-pin resistor from a 2-pin capacitor, so those are being
done by hand.
Parts:
- J2: symbol kml-custom:WAGO_2606-1104_010-000 -> KMLib_Connectors:2606-1104_010-000_Wago
- U1: symbol SparkFun-DiscreteSemi:AP63205 -> KMLib_IC_Power:AP63205WU-7_Buck_Regulator
Changed lines of the file:
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@@
 	)
 	(symbol
-		(lib_id "SparkFun-DiscreteSemi:AP63205")
+		(lib_id "KMLib_IC_Power:AP63205WU-7_Buck_Regulator")
 		(at 35.56 73.66 0)
 		(unit 1)
@@
 	)
 	(symbol
-		(lib_id "kml-custom:WAGO_2606-1104_010-000")
+		(lib_id "KMLib_Connectors:2606-1104_010-000_Wago")
 		(at 168.91 106.68 0)
 		(mirror x)

Commit message: fix(hw): re-point stale library nicknames
These parts exist in KiCad-Master-Lib; the boards referenced libraries that no
longer exist (kml-custom, KML-Custom, and SparkFun libraries that never
contained the part) or names the library has since changed.

KiCad embeds footprint geometry in the .kicad_pcb, so the boards rendered and
fabricated correctly and the rot stayed invisible -- it only surfaces on
update-from-library, or when a generator tries to resolve a nickname.

Nickname/name only. No geometry is changed:

  SparkFun-LED:WS2812-5050-4PIN -> KMLib_IC_SMD:WS2812-5050-4PIN
  kml-custom:Thermal Pad -> KMLib_Mounting:Thermal_Pad
  kml-custom:WS2812-5050-4PIN -> KMLib_IC_SMD:WS2812-5050-4PIN

Only references that failed to resolve were touched. Generic parts (<=4 pins)
and KiCad *-rescue libraries are deliberately excluded: fingerprint matching
cannot distinguish a 2-pin resistor from a 2-pin capacitor, so those are being
done by hand.
Parts:
- D1: footprint kml-custom:WS2812-5050-4PIN -> KMLib_IC_SMD:WS2812-5050-4PIN
- HS1: footprint kml-custom:Thermal Pad -> KMLib_Mounting:Thermal_Pad
Changed lines of the file:
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@@
 			)
 		)
-		(property "Footprint" "kml-custom:WS2812-5050-4PIN"
+		(property "Footprint" "KMLib_IC_SMD:WS2812-5050-4PIN"
 			(at 13.97 49.53 0)
 			(hide yes)
@@
 			)
 		)
-		(property "Footprint" "kml-custom:Thermal Pad"
+		(property "Footprint" "KMLib_Mounting:Thermal_Pad"
 			(at 35.8648 97.79 0)
 			(hide yes)
