File: hardware_new/BREAD_Slice.kicad_sch (KiCad schematic)
At the start: 23 parts, among them J1 I2C_01x04, J2 Conn_01x10_Female, J3 Screw_Terminal_01x02, J4 Screw_Terminal_01x02, J5 Screw_Terminal_01x02, J6 Screw_Terminal_01x02, U2 ACS723xMATR-10AB, U3 ACS723xMATR-10AB, U4 ACS723xMATR-10AB, U5 ACS723xMATR-10AB

Commit message: updated to latest template
Parts:
- removed J1: I2C_01x04, Connector_JST:JST_SH_SM04B-SRSS-TB_1x04-1MP_P1.00mm_Horizontal, symbol SparkFun-Connector:I2C_01x04
- removed J6: Screw_Terminal_01x02, CRx:Pheonix Conn Term TDPT 4 2-SP-6,35-ZB, symbol Connector:Screw_Terminal_01x02
- added J2: Screw_Terminal_01x02, CRx:Pheonix Conn Term TDPT 4 2-SP-6,35-ZB, symbol Connector:Screw_Terminal_01x02
- renumbered J2 to J1
Connections:
- net D7: now reaches A1.10 (D7)
- net D8: now reaches A1.11 (D8)
- net D9: now reaches A1.12 (D9)
- net D10: now reaches A1.13 (D10)
- net D11: now reaches A1.14 (D11)
- net D12: now reaches A1.15 (D12)
- net D13: now reaches A1.16 (D13)
- net AREF: now reaches A1.18 (AREF)
- net A6: now reaches A1.25 (A6)
- net A7: now reaches A1.26 (A7)
- net RESET: now reaches A1.28 (~{RESET})
- net D6: now reaches A1.9 (D6)
- net at U4.1 (IP+), U4.2 (IP+), U4.3 (IP+)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: now also J4.2 (Pin_2); no longer J5.2 (Pin_2)
- net at U4.5 (IP-), U4.6 (IP-), U4.7 (IP-)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: now also J4.1 (Pin_1); no longer J5.1 (Pin_1)
- net at U3.5 (IP-), U3.6 (IP-), U3.7 (IP-)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: now also J3.1 (Pin_1); no longer J4.1 (Pin_1)
- net at U3.1 (IP+), U3.2 (IP+), U3.3 (IP+)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: now also J3.2 (Pin_2); no longer J4.2 (Pin_2)
- net at U5.5 (IP-), U5.6 (IP-), U5.7 (IP-)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: now also J5.1 (Pin_1)
- net at U5.1 (IP+), U5.2 (IP+), U5.3 (IP+)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: now also J5.2 (Pin_2)
- net at U2.5 (IP-), U2.6 (IP-), U2.7 (IP-)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: now also J2.1 (Pin_1); no longer J3.1 (Pin_1)
- net at U2.1 (IP+), U2.2 (IP+), U2.3 (IP+)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: now also J2.2 (Pin_2); no longer J3.2 (Pin_2)
- no-connect marks 18 -> 6
Other:
- moved on the sheet: H1, H2, H3, H4
