File: hardware-2layer/isolated_ac_voltage_sensor.kicad_sch (KiCad schematic)
At the start: 17 parts, among them U10 MCP4161-xxxx-P, U5 LM358

Commit message: final schematic done before split to ac dc
Parts:
- added RL1: R_load, symbol Device:R_US
- R1: value 820k 1W -> 125k 1W
- renumbered U10 to U2, U5 to U3
Connections:
- no-connect marks 0 -> 3
Other:
- note added: "Lowest AC Regularly Used R_burden = 100ohm I_secnd = 0.072mA (@9VAC) V_burden = R_burden * I_secnd = 7.2mV"
- note added: "Lowest AC Regularly Used R_line = 125000ohm V_line = 9V I_prim = V_line / R_line = 0.072mA"
- note added: "Midsupply bias required for both as we have no negative supply rails in this design"
- note added: "Typical North America AC R_line = 125000ohm V_line = 120V I_prim = V_line / R_line = 0.96mA"
- note added: "max 2VAC @10% = 2v * 0.1 = 0.2V typ. 0.96VAC @ 25% = 0.96V * 0.25 = 0.24V min 0.05VAC @ 100% = 0.05 * 1 = 0.05V"
- note added: "max at max atten. 0.5V to 4.5V @10% = (0.5V to 4.5V) * 0.1 = 0.05V to 0.45V typ. at part. atten. 1.54V to 3.46V @25% = (1.54V to 3.46V) * 0.25 = 0.385 V to 0.865V min at min atten. 2.45V to 2.55V @100% = (2.45V to 2.55V) * 0.1 = 2.45V to 2.55V"
- note added: "output max (200mV) = 2.5V -/+2V = 0.5V to 4.5V output typ. (96mV) = 2.5V -/+0.96V = 1.54V to 3.46V output min (7mV) = 2.5V -/+0.07V = 2.43V to 2.57V"
- note added: "output max in at max attenuation: 0.2V * 10 = 2V final = 0.5V to 4.5V output typ. in at part attenuation 0.24V * 10 = 2.4V final = 0.1V to 4.9V output min at min attenuation: 0.05V * 10 = 0.5V final = 2V to 3V"
- note removed: "Lowest AC Typically Used R_burden = 100ohm I_secnd = 0.072mA (@9VAC) V_burden = R_burden * I_secnd = 7.2mV"
- note removed: "Lowest AC Typically Used R_line = 125000ohm V_line = 9V I_prim = V_line / R_line = 0.072mA"
- note removed: "North America AC R_line = 125000ohm V_line = 120V I_prim = V_line / R_line = 0.96mA"
- note removed: "max 2V @10% = 2v * 0.1 = 0.2V min 0.05V @ 100% = 0.05 * 1 = 0.05V"
- note removed: "max at max atten. 0.5V - 4.5V @10% = (0.5V - 4.5V) * 0.1 = 0.05V - 0.45V min at min atten. 2.45V - 2.55V @100% = (2.45V - 2.55V) * 0.1 = 2.45V - 2.55V"
- note removed: "output max (200mV) = 2.5V +/-2V = 0.5V - 4.5V output min (5mV) = 2.5V +/-0.05V = 2.45V - 2.55V"
- note removed: "output max in at max attenuation: 0.2V x10 = 2V final = 0.5V - 4.5V output min at min attenuation: 0.05V x10 = 0.5V final = 2V - 3V"
- moved on the sheet: C5, C6, C7, C8, R1, R10, R2, R3, R4, R5, R6, R7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
